File: PCB_project/IO.kicad_sch (KiCad schematic)
At the start: 16 parts, among them J7 Conn_01x02_Male, J8 BM06B-GHS-TBT(LF)(SN), Q1 AO3400A

Commit message: Schematic updated
Other:
- title: KP-PTR -> KP-PTR project - PTR_mini
Changed lines of the file:
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@@
 	(paper "A4")
 	(title_block
-		(title "KP-PTR")
-		(date "2023-12-10")
-		(rev "1.1")
+		(title "KP-PTR project - PTR_mini")
+		(date "2026-09-17")
+		(rev "1.0")
 		(company "Polskie Towarzystwo Rakietowe")
 		(comment 1 "bartekM, FlyingBanana, Kretu, Red Labs, Stachu M, U.S. air force i inni")

Commit message: + USB connector changed to SMD
+ igniters connectors changed to single 6 pin connector
+ buzzer selected
+ crystal changed to TCXO (experimental)
+ JLC production files generated
Parts:
- added R44: 1k, Resistor_SMD:R_0402_1005Metric, symbol Device:R
- LS1: value CBT-09427-SMT -> GMD0955YB-3V2700
Connections:
- net +3V3: now also R44.1
- net at D14.2 (A), LS1.2 (-), Q1.3 (D): now also R44.2
Other:
- moved on the sheet: D14
Changed lines of the file:
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@@
+	)
+	(junction
+		(at 243.84 76.2)
+		(diameter 0)
+		(color 0 0 0 0)
 	)
 	(junction
@@
 		(color 0 0 0 0)
 	)
+	(junction
+		(at 243.84 88.9)
+		(diameter 0)
+		(color 0 0 0 0)
+	)
 	(no_connect
 		(at 166.37 29.21)
@@
 	(wire
 		(pts
+			(xy 243.84 76.2) (xy 251.46 76.2)
+		)
+		(stroke
+			(width 0)
+			(type default)
+		)
+	)
+	(wire
+		(pts
 			(xy 251.46 87.63) (xy 251.46 88.9)
 		)
@@
 		)
 	)
+	(wire
+		(pts
+			(xy 243.84 76.2) (xy 243.84 78.74)
+		)
+		(stroke
+			(width 0)
+			(type default)
+		)
+	)
 	(polyline
 		(pts
@@
 	(wire
 		(pts
-			(xy 245.11 86.36) (xy 245.11 88.9)
+			(xy 238.76 86.36) (xy 238.76 88.9)
+		)
+		(stroke
+			(width 0)
+			(type default)
+		)
+	)
+	(wire
+		(pts
+			(xy 243.84 88.9) (xy 251.46 88.9)
 		)
 		(stroke
@@
 	(wire
 		(pts
-			(xy 245.11 88.9) (xy 251.46 88.9)
+			(xy 238.76 88.9) (xy 243.84 88.9)
 		)
 		(stroke
@@
 	(wire
 		(pts
-			(xy 245.11 78.74) (xy 245.11 76.2)
+			(xy 238.76 78.74) (xy 238.76 76.2)
 		)
 		(stroke
@@
 	(wire
 		(pts
-			(xy 245.11 76.2) (xy 251.46 76.2)
+			(xy 238.76 76.2) (xy 243.84 76.2)
 		)
 		(stroke
@@
 			(width 0)
 			(type dash)
+		)
+	)
+	(wire
+		(pts
+			(xy 243.84 86.36) (xy 243.84 88.9)
+		)
+		(stroke
+			(width 0)
+			(type default)
 		)
 	)
@@
 		(fields_autoplaced yes)
 		(property "Reference" "LS1"
-			(at 255.27 80.7376 0)
+			(at 255.27 81.1542 0)
 			(show_name no)
 			(do_not_autoplace no)
@@
 			)
 		)
-		(property "Value" "CBT-09427-SMT"
-			(at 255.27 83.2776 0)
+		(property "Value" "GMD0955YB-3V2700"
+			(at 255.27 83.6942 0)
 			(show_name no)
 			(do_not_autoplace no)
@@
 				(path "/9538e4ed-27e6-4c37-b989-9859dc0d49e8/68d9bec4-a8fa-482b-99d8-a42578238d37"
 					(reference "LS1")
+					(unit 1)
+				)
+			)
+		)
+	)
+	(symbol
+		(lib_id "Device:R")
+		(at 243.84 82.55 0)
+		(unit 1)
+		(body_style 1)
+		(exclude_from_sim no)
+		(in_bom yes)
+		(on_board yes)
+		(in_pos_files yes)
+		(dnp no)
+		(property "Reference" "R44"
+			(at 241.3 83.82 90)
+			(show_name no)
+			(do_not_autoplace no)
+			(effects
+				(font
+					(size 1.27 1.27)
+				)
+			)
+		)
+		(property "Value" "1k"
+			(at 246.38 83.82 90)
+			(show_name no)
+			(do_not_autoplace no)
+			(effects
+				(font
+					(size 1.27 1.27)
+				)
+			)
+		)
+		(property "Footprint" "Resistor_SMD:R_0402_1005Metric"
+			(at 242.062 82.55 90)
+			(hide yes)
+			(show_name no)
+			(do_not_autoplace no)
+			(effects
+				(font
+					(size 1.27 1.27)
+				)
+			)
+		)
+		(property "Datasheet" ""
+			(at 243.84 82.55 0)
+			(hide yes)
+			(show_name no)
+			(do_not_autoplace no)
+			(effects
+				(font
+					(size 1.27 1.27)
+				)
+			)
+		)
+		(property "Description" ""
+			(at 243.84 82.55 0)
+			(show_name no)
+			(do_not_autoplace no)
+			(effects
+				(font
+					(size 1.27 1.27)
+				)
+			)
+		)
+		(pin "1"
+		)
+		(pin "2"
+		)
+		(instances
+			(project "kp-ptr"
+				(path "/9538e4ed-27e6-4c37-b989-9859dc0d49e8/68d9bec4-a8fa-482b-99d8-a42578238d37"
+					(reference "R44")
 					(unit 1)
 				)
@@
 	(symbol
 		(lib_id "Diode:1N4148")
-		(at 245.11 82.55 270)
+		(at 238.76 82.55 270)
 		(unit 1)
 		(body_style 1)
@@
 		(dnp no)
 		(property "Reference" "D14"
-			(at 234.95 81.28 90)
+			(at 228.6 81.28 90)
 			(show_name no)
 			(do_not_autoplace no)
@@
 		)
 		(property "Value" "B5819W SL"
-			(at 232.41 84.074 90)
+			(at 226.06 84.074 90)
 			(show_name no)
 			(do_not_autoplace no)
@@
 		)
 		(property "Footprint" "Diode_SMD:D_SOD-123"
-			(at 240.665 82.55 0)
+			(at 234.315 82.55 0)
 			(hide yes)
 			(show_name no)
@@
 		)
 		(property "Datasheet" "https://assets.nexperia.com/documents/data-sheet/1N4148_1N4448.pdf"
-			(at 245.11 82.55 0)
+			(at 238.76 82.55 0)
 			(hide yes)
 			(show_name no)
@@
 		)
 		(property "Description" ""
-			(at 245.11 82.55 0)
-			(show_name no)
-			(do_not_autoplace no)
+			(at 238.76 82.55 0)
+			(show_name no)
+			(do_not_autoplace no)
