File: PCB_project/sensors.kicad_sch (KiCad schematic)
At the start: 14 parts, among them U2 MS560702BA03-50, U3 H3LIS331, U4 LSM6DSV32

Commit message: Schematic updated
Other:
- title: KP-PTR -> KP-PTR project - PTR_mini
Changed lines of the file:
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@@
 	(paper "A4")
 	(title_block
-		(title "KP-PTR")
-		(date "2023-12-10")
-		(rev "1.1")
+		(title "KP-PTR project - PTR_mini")
+		(date "2026-09-17")
+		(rev "1.0")
 		(company "Polskie Towarzystwo Rakietowe")
 		(comment 1 "bartekM, FlyingBanana, Kretu, Red Labs, Stachu M, U.S. air force i inni")

Commit message: + USB connector changed to SMD
+ igniters connectors changed to single 6 pin connector
+ buzzer selected
+ crystal changed to TCXO (experimental)
+ JLC production files generated
Parts:
- C18, C21: footprint Capacitor_SMD:C_0402_1005Metric -> Capacitor_SMD:C_0603_1608Metric
Changed lines of the file:
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@@
 			)
 		)
-		(property "Footprint" "Capacitor_SMD:C_0402_1005Metric"
+		(property "Footprint" "Capacitor_SMD:C_0603_1608Metric"
 			(at 96.2152 78.105 0)
 			(hide yes)
@@
 			)
 		)
-		(property "Footprint" "Capacitor_SMD:C_0402_1005Metric"
+		(property "Footprint" "Capacitor_SMD:C_0603_1608Metric"
 			(at 162.2552 78.74 0)
 			(hide yes)
