File: PTR_mini_pcb/PTR_mini_pcb.kicad_pcb (KiCad board)
At the start: 4 copper layers, 25 x 74 mm, 140 parts, among them IC1 TPS62142, J1 ESP32_PROG_CON, J14 Molex 104031-0811, J2 Conn_01x02, J3 67996-104HLF, J4 USB4105-GF-A-120, J5 DB125-3.5-6P-GN-S, J7 Conn_01x02_Male, J8 BM06B-GHS-TBT(LF)(SN), Q1 AO3400A, Q12 AO3400A, Q2 AO3401A, Q4 AO3401A, Q6 AO3400A, Q7 AO3400A, Q8 AO3401A, U1 ESP32-S3FN8, U10 LDL1117S50R, U11 USBLC6-2SC6-ES, U13 W25Q256, U2 MS560702BA03-50, U3 H3LIS331, U4 LSM6DSV32, Y2 X1G0054210307

Commit message: SPI Flash moved to different SPI lines
Connections:
- net SPI2_CS_FLASH renamed SPI_CS_FLASH
- U13 pad 2: SPI2_MISO -> SPI_MISO
- U13 pad 5: SPI2_MOSI -> SPI_MOSI
- U13 pad 6: SPI2_SCK -> SPI_SCK
Routing:
- net SPI_MOSI: track 32.0 -> 46.6 mm, vias 2 -> 3
- net SPI_MISO: track 30.1 -> 42.3 mm, vias 4 -> 5
- net SPI_SCK: track 36.6 -> 48.5 mm, vias 4 -> 6
- net SPI2_MOSI: track 16.2 -> 6.03 mm, vias 2 -> 1
- net SPI2_SCK: track 16.2 -> 6.81 mm, vias 3 -> 1
- net SPI2_MISO: track 14.7 -> 8.45 mm, vias 2 -> 1
- net LSM_INT: track 31.0 -> 31.6 mm

Commit message: TCXO replaced with 10ppm crystal
Parts:
- removed C24: 100nF, Capacitor_SMD:C_0402_1005Metric
- removed C25, C26: 10nF, Capacitor_SMD:C_0402_1005Metric
- removed Y2: X1G0054210307, Oscillator:Oscillator_SMD_SeikoEpson_TG2520SMN-xxx-xxxxxx-4Pin_2.5x2.0mm
- added C10: 15pF, Capacitor_SMD:C_0402_1005Metric, B.Cu at (14.2, 20.7)
- added C9: 15pF, Capacitor_SMD:C_0402_1005Metric, B.Cu at (16.5, 22.4)
- added L3: 24nH, Inductor_SMD:L_0402_1005Metric, B.Cu at (13.8, 24.4)
- added Y3: XTM20040000FT00351001, Crystal:Crystal_SMD_2016-4Pin_2.0x1.6mm, B.Cu at (14.5, 22.3)
Routing:
- net Net-(C9-Pad2): track 0.00 -> 3.56 mm
- net Net-(Y2-OUT): track 3.19 -> 0.00 mm
- net Net-(U1-XTAL_N): track 4.16 -> 6.70 mm
- net +3V3: track 92.3 -> 90.2 mm, vias 34 -> 33
- net LED: track 33.0 -> 31.8 mm
- net Net-(D10-DOUT): track 62.4 -> 63.4 mm
- net Earth: vias 95 -> 98

Commit message: +Flash model changed
+new step models
Parts:
- U13: value W25Q256 -> GD25Q256EWIGR
Routing:
- net USB_DP: track 29.8 -> 27.8 mm
- net Net-(J4-D+-PadA6): track 5.20 -> 6.91 mm
- net VBUS: track 42.7 -> 41.8 mm
- net Earth: track 48.0 -> 47.8 mm, vias 98 -> 109
